File: Hardware/schematic_tsc.sch (EAGLE design)
At the start: 105 parts, among them IC1 BQ25180YBGR, IC2 DRV2605YZFR, IC3 BMA423, IC9 RT6160AWSC, J1 503480-2400, J2 TC2030-IDC, J4 KH-TYPE-C-16P, Q1 20V/4.2A/52mΩ/1.4W, Q3 SI1308EDL-T1-GE3, U1 NRF52840_QF, U3 MAX17048G+T10, X1 32MHz, X2 32.768kHz

Commit message: New files added
Parts:
- C16: value 47µF -> 47nF; device InkTime_v5:NORDIC_NRF_3_CAPACITOR_0402_L -> InkTime_v5:NORDIC_NRF_3_CAPACITOR_0201_L
- L1: device InkTime_v5:NORDIC_NRF_2_INDUCTOR_0201_N -> InkTime_v5:NORDIC_NRF_2_INDUCTOR_0402_L
- L2: value 10µH -> 10uH; device InkTime_v5:NORDIC_NRF_2_INDUCTOR_0201_N -> InkTime_v5:NORDIC_NRF_2_INDUCTOR_0603_L
- L3: value 15µH -> 15nH; device InkTime_v5:NORDIC_NRF_2_INDUCTOR_0201_N -> InkTime_v5:NORDIC_NRF_2_INDUCTOR_0402_L
- L5: device InkTime_v5:NORDIC_NRF_2_INDUCTOR_0201_N -> InkTime_v5:ESP32_C6_LIBRARY_2_744043680IND_4828-WE-TPC_WRE
- R1_USB, R2_USB: value 5k1 -> 5K1
- R5, R7, R8: value 10k -> 10K
- renumbered D3 to D1, SW_DN to SW3
Connections:
- removed net 3V3/1.7D: C34.2, IC2.VDD, Q1.S, R5.2, R_PWR_EPD.2
- removed net 3V3/2.4A: C12.1, C14.1, C19.1, C25.1, C33.1, C6.1, C7.1, C8.1, IC3.CSB, IC3.VDD, IC3.VDDIO, IC9.VOUT_1, IC9.VOUT_2, J2.1, R17.1, R18.1, TP_3.3V.TP, TP_3V3.TP, U1.VDD@A22, U1.VDD@AD14, U1.VDD@AD23, U1.VDD@B1, U1.VDD@W1, U1.VDDH@Y2
- removed net P0.04: U1.P0.04/AIN2@J1
- removed net P0.09: U1.P0.09/NFC1@L24
- removed net P0.19: U1.P0.19@AC15
- removed net P0.20: U1.P0.20@AD16
- removed net P0.21: U1.P0.21@AC17
- removed net P0.22: U1.P0.22@AD18
- removed net P0.23: U1.P0.23@AC19
- removed net P0.24: U1.P0.24@AD20
- removed net P0.25: U1.P0.25@AC21
- removed net P0.26: U1.P0.26@G1
- removed net P0.27: U1.P0.27@H2
- removed net P0.28: U1.P0.28/AIN4@B11
- removed net P0.29: U1.P0.29/AIN5@A10
- removed net P0.30: U1.P0.30/AIN6@B9
- removed net P0.31: U1.P0.31/AIN7@A8
- removed net P1.03: U1.P1.03@V23
- removed net P1.04: U1.P1.04@U24
- removed net P1.05: U1.P1.05@T23
- removed net P1.06: U1.P1.06@R24
- removed net P1.07: U1.P1.07@P23
- removed net P1.09: U1.P1.09@R1
- removed net P1.10: U1.P1.10@A20
- removed net P1.11: U1.P1.11@B19
- removed net P1.12: U1.P1.12@B17
- removed net P1.13: U1.P1.13@A16
- removed net P1.14: U1.P1.14@B15
- removed net P1.15: U1.P1.15@A14
- removed net SCL/1.4C: IC2.SCL, U3.SCL
- removed net SCL/2.4C: IC1.SCL, IC3.SCX, R17.2, R4.1, TP_SCL.TP, U1.P0.07@M2
- removed net SDA/1.4C: IC2.SDA, U3.SDA
- removed net SDA/2.4C: IC1.SDA, IC3.SDX, R18.2, R2.1, TP_SDA.TP, U1.P0.06@L1
- removed net VBAT/1.2A: C27.2, TP_VBAT.TP, U3.CELL, U3.VDD
- removed net VBAT/2.5C: C37.2, IC1.BAT
- removed net VBUS/1.5D: C42.1, C43.1, D1.VBUS, J4.VBUS
- removed net VBUS/2.6D: C21.1, C38.2, IC1.IN, U1.VBUS@AD2
- new net 3V3: C12.1, C14.1, C19.1, C25.1, C33.1, C34.2, C6.1, C7.1, C8.1, IC2.VDD, IC3.CSB, IC3.VDD, IC3.VDDIO, IC9.VOUT_1, IC9.VOUT_2, J2.1, Q1.S, R17.1, R18.1, R5.2, R_PWR_EPD.2, TP_3.3V.TP, TP_3V3.TP, U1.VDD@A22, U1.VDD@AD14, U1.VDD@AD23, U1.VDD@B1, U1.VDD@W1, U1.VDDH@Y2
- new net SCL: IC1.SCL, IC2.SCL, IC3.SCX, R17.2, R4.1, TP_SCL.TP, U1.P0.07@M2, U3.SCL
- new net SDA: IC1.SDA, IC2.SDA, IC3.SDX, R18.2, R2.1, TP_SDA.TP, U1.P0.06@L1, U3.SDA
- new net VBAT: C27.2, C37.2, IC1.BAT, TP_VBAT.TP, U3.CELL, U3.VDD
- new net VBUS: C21.1, C38.2, C42.1, C43.1, D1.VBUS, IC1.IN, J4.VBUS, U1.VBUS@AD2
- net DEC4_6: now also L3.1; no longer L3.2
- net EPD_3V3: now also L5.2; no longer L5.1
- net N$10: now also L2.2; no longer L2.1
- net N$11: now also L2.1, L3.2; no longer L2.2, L3.1
- net N$8: now also L5.1; no longer L5.2
Other:
- note added: "Placeholder"
- moved on the sheet: C27, L2, L3, TP_BAT_GND, TP_VBAT, U3
